File: PCB/aniweather.kicad_pcb (KiCad board)
At the start: 2 copper layers, 0 parts

Commit message: Saber plus PCB start
Parts:
- added BT1: Battery_Cell, TestPoint:TestPoint_2Pads_Pitch5.08mm_Drill1.3mm, F.Cu at (130.9, 87.0)
- added C1: Tiny, Capacitor_THT:C_Disc_D5.0mm_W2.5mm_P2.50mm, F.Cu at (156.5, 78.5)
- added C2: Tiny, Capacitor_THT:C_Disc_D5.0mm_W2.5mm_P2.50mm, F.Cu at (156.5, 82.5)
- added C3: Tiny, Capacitor_THT:C_Disc_D5.0mm_W2.5mm_P2.50mm, F.Cu at (156.5, 86.6)
- added C4: Tiny, Capacitor_THT:C_Disc_D5.0mm_W2.5mm_P2.50mm, F.Cu at (192.2, 106.5)
- added G: LOGO, LOGO, F.Cu at (136.7, 39.1)
- added G: LOGO, LOGO, B.Cu at (48.5, 71.0)
- added H1: MountingHole, MountingHole:MountingHole_3.2mm_M3, F.Cu at (222.0, 50.0)
- added H2: MountingHole, MountingHole:MountingHole_3.2mm_M3, F.Cu at (175.0, 50.0)
- added H3: MountingHole, MountingHole:MountingHole_3.2mm_M3, F.Cu at (175.0, 117.0)
- added H4: MountingHole, MountingHole:MountingHole_3.2mm_M3, F.Cu at (222.0, 117.0)
- added R1: 10, Resistor_THT:R_Axial_DIN0207_L6.3mm_D2.5mm_P10.16mm_Horizontal, F.Cu at (197.2, 114.1)
- added SW1: SW_DIP_x01, Button_Switch_THT:SW_DIP_SPSTx01_Slide_9.78x4.72mm_W7.62mm_P2.54mm, F.Cu at (120.0, 81.5)
- added SW2: SW_Push, Button_Switch_THT:SW_PUSH_6mm, F.Cu at (120.1, 86.7)
- added U1: ~, asylum:ST7735, F.Cu at (198.5, 83.5)
- added U2: ~, asylum:WEMOS_C1_mini, F.Cu at (207.3, 89.6)
- added U3: ~, asylum:TP4056, F.Cu at (130.2, 82.0)
Routing:
- net +3.3V: track 0.00 -> 28.2 mm
- net SDA: track 0.00 -> 17.4 mm
- net SCK: track 0.00 -> 17.4 mm
- net AO: track 0.00 -> 16.4 mm
- net RESET: track 0.00 -> 15.5 mm
- net CS_LCD: track 0.00 -> 15.3 mm
- net Net-(U1-LED): track 0.00 -> 4.10 mm
- net GND: vias 0 -> 80
- added copper zone on B.Cu, net GND
- added copper zone on F.Cu, net GND
Other:
- board outline added: 55 x 75 mm

Commit message: V1.0
Parts:
- added C5: 0.1uF, Capacitor_THT:C_Disc_D5.0mm_W2.5mm_P2.50mm, B.Cu at (126.5, 102.0)
- added C6: 10uF, Capacitor_THT:C_Disc_D5.0mm_W2.5mm_P2.50mm, B.Cu at (118.0, 100.8)
- added C7: 10uF, Capacitor_THT:C_Disc_D5.0mm_W2.5mm_P2.50mm, B.Cu at (118.0, 114.8)
- added C8: 10uF, Capacitor_THT:C_Disc_D5.0mm_W2.5mm_P2.50mm, B.Cu at (118.0, 110.4)
- added L1: 2.2uH, Inductor_SMD:L_1210_3225Metric, B.Cu at (116.8, 105.3)
- added R2: 100, Resistor_THT:R_Axial_DIN0207_L6.3mm_D2.5mm_P10.16mm_Horizontal, B.Cu at (128.1, 97.8)
- added U5: TPS63001, Package_SON:Texas_DRC0010J_ThermalVias, B.Cu at (120.5, 105.4)
- BT1, U3: moved to B.Cu
- moved G 94.4 mm to (140.1, 94.2)
- moved SW1 64.9 mm to (163.9, 129.2), turned to 90 degrees
- moved C4 63.2 mm to (131.4, 123.9), turned to 0 degrees
- moved H1 60.8 mm to (163.7, 67.4)
- moved H4 60.8 mm to (163.7, 134.4)
- moved R1 60.8 mm to (138.9, 131.5)
- moved U1 60.8 mm to (140.2, 100.9)
- moved H2 60.8 mm to (116.7, 67.4)
- moved H3 60.8 mm to (116.7, 134.4)
- moved U2 60.8 mm to (149.0, 107.0)
- moved C1 58.5 mm to (127.9, 129.5), turned to 90 degrees
- moved SW2 57.3 mm to (157.9, 129.7), turned to -90 degrees
- moved G 56.8 mm to (139.7, 95.8)
- moved C2 47.9 mm to (128.4, 121.3), turned to -90 degrees
- moved BT1 22.1 mm to (138.4, 66.2)
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Connections:
- C3 pad 1: GND -> Net-(BT1-+)
- C3 pad 2: +3.3V -> Net-(BT1--)
- C4 pad 1: GND -> +3.3V
- C4 pad 2: +3.3V -> GND
- SW2 pad 2: unconnected-(SW2-Pad2) -> Net-(U2-A5)
- U2 pad 0: AO -> SDA
- U2 pad 1: RESET -> AO
- U2 pad 10: SD_MOSI -> SD_CS
- U2 pad 2: CS_LCD -> RESET
- U2 pad 3: unconnected-(U2-A3-Pad3) -> CS_LCD
- U2 pad 4: SDA -> SCK
- U2 pad 5: SCK -> Net-(U2-A5)
- U2 pad 6: unconnected-(U2-Pad6) -> SD_SCK
- U2 pad 7: unconnected-(U2-7/RGB_LED-Pad7) -> SD_MISO
- U2 pad 8: unconnected-(U2-Pad8) -> SD_MOSI
Routing:
- net +3.3V: track 28.2 -> 108.6 mm
- net Net-(BT1-+): track 0.00 -> 33.1 mm
- net Net-(BT1--): track 0.00 -> 28.6 mm
- net Net-(U3-OUT+): track 0.00 -> 26.6 mm
- net SD_CS: track 0.00 -> 25.8 mm
- net SD_MISO: track 0.00 -> 25.3 mm
- net SD_SCK: track 0.00 -> 25.3 mm
- net SD_MOSI: track 0.00 -> 25.3 mm
- net GND: track 0.00 -> 22.4 mm, vias 80 -> 88
- net Net-(U5-EN): track 0.00 -> 17.8 mm
- net Net-(U2-A5): track 0.00 -> 12.6 mm
- net Net-(U2-3.3V): track 0.00 -> 6.98 mm
- net AO: track 16.4 -> 13.3 mm
- net SDA: track 17.4 -> 14.7 mm
- net RESET: track 15.5 -> 12.9 mm
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- added copper zone on B.Cu, net +3.3V
- added copper zone on B.Cu, net Net-(U3-OUT+)
- added copper zone on B.Cu, net Net-(U5-L1)
- added copper zone on B.Cu, net Net-(U5-L2)

Commit message: V1.0 rev 1
Parts:
- moved U3 0.30 mm to (126.0, 84.9)
Routing:
- net GND: track 22.4 -> 33.1 mm, vias 88 -> 86
- net Net-(BT1-+): track 33.1 -> 38.0 mm
- net Net-(BT1--): track 28.6 -> 32.8 mm

Commit message: Fix some small issues
Parts:
- removed G (x2): LOGO, LOGO
- added C9: Tiny, Capacitor_THT:C_Disc_D5.0mm_W2.5mm_P2.50mm, B.Cu at (158.4, 120.9)
- added G1: LOGO, LOGO, B.Cu at (70.1, 95.6)
- added G2: LOGO, LOGO, F.Cu at (70.1, 95.6)
- added R3: 100k, Resistor_THT:R_Axial_DIN0207_L6.3mm_D2.5mm_P10.16mm_Horizontal, F.Cu at (166.4, 126.3)
- U3: moved to F.Cu
- moved SW1 55.8 mm to (117.7, 98.0), turned to -90 degrees
- moved C8 13.3 mm to (118.8, 123.7), turned to 180 degrees
- moved U5 11.2 mm to (120.1, 116.7)
- moved C5 11.2 mm to (126.2, 113.2)
- moved C6 11.2 mm to (117.6, 112.0)
- moved L1 11.2 mm to (116.4, 116.5)
- moved R2 11.2 mm to (127.8, 109.0)
- moved C7 5.83 mm to (118.8, 120.6), turned to 180 degrees
- moved BT1 5.08 mm to (143.5, 66.2), turned to 180 degrees
- moved C3 2.50 mm to (136.2, 83.7), turned to -90 degrees
- turned U3 to 90 degrees
Connections:
- C6 pad 1: Net-(U3-OUT+) -> Net-(U5-VIN)
- R2 pad 2: Net-(U3-OUT+) -> Net-(U5-VIN)
- SW1 pad 1: +3.3V -> Net-(U3-OUT+)
- SW1 pad 2: Net-(U2-3.3V) -> Net-(U5-VIN)
- U2 pad 11: +3.3V -> unconnected-(U2-EN-Pad11)
- U2 pad 12: Net-(U2-3.3V) -> +3.3V
- U3 pad 4: BAT_IN+ -> unconnected-(U3-IN+-Pad4)
- U3 pad 5: BAT_IN- -> unconnected-(U3-IN--Pad5)
- U5 pad 5: Net-(U3-OUT+) -> Net-(U5-VIN)
Routing:
- net +3.3V: track 108.6 -> 89.2 mm
- net GND: track 33.1 -> 23.3 mm, vias 86 -> 72
- net Net-(U5-VIN): track 0.00 -> 9.54 mm
- net Net-(BT1-+): track 38.0 -> 29.2 mm
- net Net-(U2-3.3V): track 6.98 -> 0.00 mm
- net Net-(U2-A5): track 12.6 -> 19.1 mm
- net Net-(U3-OUT+): track 26.9 -> 29.3 mm
- net Net-(BT1--): track 32.8 -> 35.1 mm
- net Net-(U5-L1): track 0.00 -> 0.68 mm
- net Net-(U5-L2): track 0.00 -> 0.66 mm
- added copper zone on B.Cu, net Net-(U5-VIN)
- removed copper zone on B.Cu, net Net-(U3-OUT+)

Commit message: Bottom case
Parts:
- moved G1 70.3 mm to (140.4, 95.5)
- moved G2 70.3 mm to (140.4, 95.5)
Changed lines of the file:
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@@
 	(footprint "LOGO"
 		(layer "F.Cu")
-		(at 70.1 95.6)
+		(at 140.35115 95.527339)
 		(property "Reference" "G2"
 			(at 0 0 0)
@@
 			(size 2.2 2.2)
 			(drill 1.5)
-			(layers "F&B.Cu" "*.Mask")
+			(layers "*.Cu" "*.Mask")
 			(remove_unused_layers no)
 			(net 1 "Net-(BT1-+)")
@@
 			(size 2.2 2.2)
 			(drill 1.5)
-			(layers "F&B.Cu" "*.Mask")
+			(layers "*.Cu" "*.Mask")
 			(remove_unused_layers no)
 			(net 2 "Net-(BT1--)")
@@
 			(size 2.2 2.2)
 			(drill 1.5)
-			(layers "F&B.Cu" "*.Mask")
+			(layers "*.Cu" "*.Mask")
 			(remove_unused_layers no)
 			(net 19 "Net-(U3-OUT+)")
@@
 			(size 2.2 2.2)
 			(drill 1.5)
-			(layers "F&B.Cu" "*.Mask")
+			(layers "*.Cu" "*.Mask")
 			(remove_unused_layers no)
 			(net 15 "GND")
@@
 			(size 2.2 2.2)
 			(drill 1.5)
-			(layers "F&B.Cu" "*.Mask")
+			(layers "*.Cu" "*.Mask")
 			(remove_unused_layers no)
 			(net 21 "unconnected-(U3-IN+-Pad4)")
@@
 			(size 2.2 2.2)
 			(drill 1.5)
-			(layers "F&B.Cu" "*.Mask")
+			(layers "*.Cu" "*.Mask")
 			(remove_unused_layers no)
 			(net 20 "unconnected-(U3-IN--Pad5)")
@@
 		(model "${KIPRJMOD}/libs/asylum.pretty/C3-mini.step"
 			(offset
-				(xyz -12.7 -18.9 0.5)
+				(xyz -12.7 -18.9 3.5)
 			)
 			(scale
@@
 			(at -0.575 0)
 			(size 0.5 0.5)
-			(drill 0.3)
+			(drill 0.2)
 			(layers "F&B.Cu")
 			(remove_unused_layers no)
@@
 		(pad "11" thru_hole circle
 			(at 0 -0.95)
-			(size 0.7 0.7)
-			(drill 0.3)
+			(size 0.5 0.5)
+			(drill 0.2)
 			(layers "F&B.Cu")
 			(remove_unused_layers no)
@@
 			(at 0 0.95)
 			(size 0.5 0.5)
-			(drill 0.3)
+			(drill 0.2)
 			(layers "F&B.Cu")
 			(remove_unused_layers no)
@@
 			(at 0.575 0)
 			(size 0.5 0.5)
-			(drill 0.3)
+			(drill 0.2)
 			(layers "F&B.Cu")
 			(remove_unused_layers no)
@@
 	(footprint "LOGO"
 		(layer "B.Cu")
-		(at 70.1 95.6 180)
+		(at 140.35115 95.527339 180)
 		(property "Reference" "G1"
 			(at 0 0 0)
