File: PCB/aniweather.kicad_pcb (KiCad board)
At the start: 2 copper layers, 55 x 75 mm, 36 parts, among them SW1 SW_DIP_x01, SW2 SW_Push, SW3 SW_Push, U5 TPS63001

Commit message: Hope last rev
Parts:
- moved C2 48.1 mm to (154.2, 80.8)
Routing:
- net CS_LCD: track 43.0 -> 44.0 mm
- net GND: vias 51 -> 50
Changed lines of the file:
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@@
 		(title "Aniweather")
 		(date "2024-12-06")
-		(rev "v1.11")
+		(rev "v1.12")
 		(company "Cyao")
 		(comment 1 "Anime weather station")
@@
 		(tags "Diode DO-35_SOD27 series Axial Horizontal pin pitch 7.62mm  length 4mm diameter 2mm")
 		(property "Reference" "D1"
-			(at 3.81 -2.12 360)
+			(at 3.81 -2.12 0)
 			(layer "F.SilkS")
 			(effects
@@
 		)
 		(property "Value" "D"
-			(at 3.81 2.12 360)
+			(at 3.81 2.12 0)
 			(layer "F.Fab")
 			(effects
@@
 		)
 		(property "Footprint" ""
-			(at 0 0 360)
+			(at 0 0 0)
 			(layer "F.Fab")
 			(hide yes)
@@
 		)
 		(fp_text user "K"
-			(at 0 -1.8 360)
+			(at 0 -1.8 0)
 			(layer "F.SilkS")
 			(effects
@@
 		)
 		(fp_text user "K"
-			(at 0 -1.8 360)
+			(at 0 -1.8 0)
 			(layer "F.Fab")
 			(effects
@@
 		)
 		(fp_text user "${REFERENCE}"
-			(at 4.11 0 360)
+			(at 4.11 0 0)
 			(layer "F.Fab")
 			(effects
@@
 	(footprint "Capacitor_THT:C_Disc_D5.0mm_W2.5mm_P2.50mm"
 		(layer "F.Cu")
-		(at 128.375 121.35 -90)
+		(at 154.225 80.825 -90)
 		(descr "C, Disc series, Radial, pin pitch=2.50mm, , diameter*width=5*2.5mm^2, Capacitor, http://cdn-reichelt.de/documents/datenblatt/B300/DS_KERKO_TC.pdf")
 		(tags "C Disc series Radial pin pitch 2.50mm  diameter 5mm width 2.5mm Capacitor")
@@
 	)
 	(segment
-		(start 156.41 86.325)
-		(end 154.58 86.325)
+		(start 158.4 120.075)
+		(end 158.4 120.925)
 		(width 1.5)
 		(layer "F.Cu")
@@
 	)
 	(segment
-		(start 158.4 120.075)
-		(end 158.4 120.925)
+		(start 156.41 86.325)
+		(end 156.41 85.51)
 		(width 1.5)
 		(layer "F.Cu")
@@
 	)
 	(segment
-		(start 154.58 86.325)
-		(end 151.53 83.275)
+		(start 156.41 85.51)
+		(end 154.225 83.325)
 		(width 1.5)
 		(layer "F.Cu")
@@
 	)
 	(segment
+		(start 154.225 83.325)
+		(end 151.66 83.325)
+		(width 1.5)
+		(layer "F.Cu")
+		(net 4)
+	)
+	(segment
+		(start 151.66 83.325)
+		(end 151.61 83.275)
+		(width 1.5)
+		(layer "F.Cu")
+		(net 4)
+	)
+	(segment
 		(start 158.4 120.925)
 		(end 158.4 129.675)
@@
 	)
 	(segment
-		(start 142.75 119.875)
-		(end 142.75 119.825)
-		(width 0.5)
+		(start 146.54 95.565)
+		(end 146.54 94.385)
+		(width 0.75)
 		(layer "F.Cu")
 		(net 6)
 	)
 	(segment
-		(start 136.395 126.23)
-		(end 142.75 119.875)
-		(width 0.5)
+		(start 146.54 94.385)
+		(end 147.75 93.175)
+		(width 0.75)
 		(layer "F.Cu")
 		(net 6)
 	)
 	(segment
-		(start 143.5 100.725)
-		(end 144.9 99.325)
+		(start 142.45 116.525)
+		(end 140.7 116.525)
 		(width 0.5)
 		(layer "F.Cu")
@@
 	)
 	(segment
-		(start 146.54 95.565)
-		(end 146.54 94.385)
+		(start 147.75 93.175)
+		(end 147.75 91.175)
 		(width 0.75)
 		(layer "F.Cu")
@@
 	)
 	(segment
-		(start 146.54 94.385)
-		(end 147.75 93.175)
-		(width 0.75)
+		(start 139.725 122.9)
+		(end 136.395 126.23)
+		(width 0.5)
 		(layer "F.Cu")
 		(net 6)
 	)
 	(segment
-		(start 142.75 117.125)
-		(end 143.5 116.375)
+		(start 140.7 116.525)
+		(end 139.725 117.5)
 		(width 0.5)
 		(layer "F.Cu")
@@
 	)
 	(segment
-		(start 147.75 93.175)
-		(end 147.75 91.175)
-		(width 0.75)
+		(start 139.725 117.5)
+		(end 139.725 122.9)
+		(width 0.5)
 		(layer "F.Cu")
 		(net 6)
 	)
 	(segment
-		(start 143.5 116.375)
+		(start 144.9 99.325)
 		(end 143.5 100.725)
 		(width 0.5)
@@
 	)
 	(segment
-		(start 142.75 119.825)
-		(end 142.75 117.125)
-		(width 0.45)
+		(start 147.25 90.675)
+		(end 147.25 89.375)
+		(width 0.75)
 		(layer "F.Cu")
 		(net 6)
 	)
 	(segment
-		(start 147.25 90.675)
-		(end 147.25 89.375)
-		(width 0.75)
+		(start 143.5 115.475)
+		(end 142.45 116.525)
+		(width 0.5)
 		(layer "F.Cu")
 		(net 6)
 	)
 	(segment
-		(start 136.395 127.425)
-		(end 136.395 126.23)
+		(start 136.395 126.23)
+		(end 136.395 127.425)
 		(width 0.5)
 		(layer "F.Cu")
@@
 		(net 6)
 	)
+	(segment
+		(start 143.5 100.725)
+		(end 143.5 115.475)
+		(width 0.5)
+		(layer "F.Cu")
+		(net 6)
+	)
 	(via
 		(at 144.9 99.325)
@@
 	)
 	(via
-		(at 155.8 91.175)
+		(at 156.15 91.425)
 		(size 1)
 		(drill 0.6)
@@
 	)
 	(via
-		(at 156.775 92.55)
+		(at 156.725 93.2)
 		(size 1)
 		(drill 0.6)
@@
 		(size 1)
 		(drill 0.6)
-		(layers "F.Cu" "B.Cu")
-		(free yes)
-		(net 14)
-	)
-	(via
-		(at 145.1 90.075)
-		(size 1)
-		(drill 0.6)
